File: DC-Starter-V1/DC-Soft-Starter_NMOS/DC-Soft-Starter.sch (KiCad schematic (older format))
At the start: 58 parts

Commit message: no message
Parts:
- removed C?: CAP, symbol pspice:CAP
- removed C?: 100nF, symbol Device:C_Small
- removed D?, Rectifier: D_Bridge_+-AA, symbol Device:D_Bridge_+-AA
- removed D? (x2): D_TVS, symbol Device:D_TVS
- removed J? (x3): Conn_01x02, symbol Connector:Conn_01x02_Male
- removed Q? (x3): NMOS, Package_TO_SOT_SMD:SOT-23, symbol Transistor_FET:ZXMN2A14F
- removed R?: filter res, symbol Device:R_US
- removed R? (x3): R_US, symbol Device:R_US
- removed T? (x2): Transformer_1P_1S, symbol Device:Transformer_1P_1S
- removed s?: 1nF, symbol Device:C_Small
- added IN2: 15 VDC, Connector_Phoenix_MSTB:PhoenixContact_MSTBA_2,5_2-G_1x02_P5.00mm_Horizontal, symbol Connector:Screw_Terminal_01x02
- added J1: Screw_Terminal_01x02, Connector:Banana_Jack_2Pin, symbol Connector:Screw_Terminal_01x02
- 10kR1: renamed from 10kR; footprint (none) -> Resistor_THT:R_Axial_DIN0204_L3.6mm_D1.6mm_P2.54mm_Vertical
- 2.5_Watt1: renamed from 2.5_Watt; footprint (none) -> Resistor_THT:R_Axial_Power_L38.0mm_W9.0mm_P45.72mm
- 220R1, 220R2, 220R3, 500R1: renamed from R?; footprint (none) -> Resistor_THT:R_Axial_DIN0204_L3.6mm_D1.6mm_P5.08mm_Horizontal
- C1, C2, C6: renamed from C?; footprint (none) -> Capacitor_THT:C_Rect_L7.0mm_W2.5mm_P5.00mm
- C4: renamed from C?; footprint (none) -> Capacitor_THT:C_Rect_L9.0mm_W2.7mm_P7.50mm_MKT
- C5, C7: renamed from C?; footprint (none) -> Capacitor_THT:CP_Radial_D8.0mm_P5.00mm
- D1: renamed from D?; footprint (none) -> Diode_THT:D_A-405_P7.62mm_Horizontal; symbol Simulation_SPICE:DIODE -> DC-Soft-Starter-rescue:DIODE-Simulation_SPICE
- D2, D3, D4: renamed from D?; footprint (none) -> LED_THT:LED_D3.0mm_Clear
- D5: renamed from D?; footprint (none) -> Diode_THT:D_5W_P10.16mm_Horizontal; symbol Simulation_SPICE:DIODE -> DC-Soft-Starter-rescue:DIODE-Simulation_SPICE
- IN1: renamed from IN; footprint (none) -> Connector_Phoenix_MSTB:PhoenixContact_MSTBA_2,5_2-G_1x02_P5.00mm_Horizontal
- J2: renamed from J?; footprint (none) -> Connector:Banana_Jack_2Pin
- Q1, Q2: renamed from Q?; value IRF7799L2 -> IXFH40N30
- R1, R10, R11, R12, R2, R3, R4, R9: renamed from R?; footprint (none) -> Resistor_THT:R_Axial_DIN0204_L3.6mm_D1.6mm_P2.54mm_Vertical
- SW1, SW2: renamed from SW?; footprint (none) -> Button_Switch_THT:SW_PUSH_6mm_H9.5mm
- U5: renamed from U?; value 78M05 -> LM2575T
- s2: renamed from s; footprint (none) -> Capacitor_THT:CP_Radial_D8.0mm_P5.00mm
- gave numbers to parts that had none: 5
Connections:
- net +15V: now also IN2.2 (Pin_2); no longer A1.30 (VIN), C4.1
- net +5V: now also A1.27 (+5V), C4.1
- net GNDREF: now also SW1.4 (B), s2.1, IN2.1 (Pin_1); no longer SW1.2 (B), s2.2
- net at D1.1 (A), D5.2 (K), J2.1 (Pin_1): now also J1.2 (Pin_2)
- net at 500R1.2, U2.2: now also U3.3 (IP-), U3.4 (IP-), J1.1 (Pin_1); no longer U3.1 (IP+), U3.2 (IP+)
- net at A1.14 (D11), R3.2: now also SW1.3 (A); no longer SW1.1 (A)
- net at A1.23 (A4): now also U3.7 (VIOUT)
- net at U3.6 (FILTER): now also s2.2; no longer s2.1
- new net: Q1.1 (D), U3.1 (IP+), U3.2 (IP+)
Other:
- note removed: "1x2 Klemens\n"
- note removed: "230 VDC"
- note removed: "LIVE\n"
- note removed: "NEUTRAL\n"
